File: Salane Reboot/Paranoid/TKL/Atmega32U4/Solder Main Branch/Solder.sch (KiCad schematic (older format))
At the start: 231 parts, among them J1 Conn_01x06_Female, J2 Conn_01x04_Female, U1 ATmega32U4-MU, U2 PRTR5V0U2X, Y1 16MHz

Commit message: a
Parts:
- added R5: 300R, sanproject-keyboard-part:R_0402, symbol Device:R_Small
- renumbered C5 to C2, C2 to C3, C3 to C5, D94 to D1, D7 to D10, D8 to D11, D9 to D12, D10 to D13, D11 to D14, D12 to D15, D13 to D16, D14 to D17, D15 to D18, D16 to D19, D90 to D2, D17 to D20, D18 to D21, D19 to D22, D20 to D23, D21 to D24, D22 to D25, D23 to D26, D25 to D27, D26 to D28, D27 to D29, D93 to D3, D28 to D30, D29 to D31, D31 to D32, D32 to D33, D33 to D34, D34 to D35, D35 to D36, D1 to D4, D49 to D48, D50 to D49, D2 to D5, D51 to D50, D52 to D51, D53 to D52, D55 to D53, D56 to D54, D57 to D55, D58 to D56, D59 to D57, D61 to D58, D62 to D59, D3 to D6, D63 to D60, D64 to D61, D65 to D62, D66 to D63, D67 to D64, D68 to D65, D69 to D66, D70 to D67, D71 to D68, D72 to D69, D4 to D7, D73 to D70, D74 to D71, D75 to D72, D76 to D73, D77 to D74, D78 to D75, D79 to D76, D80 to D77, D81 to D78, D82 to D79, D5 to D8, D83 to D80, D84 to D81, D85 to D82, D24 to D83, D86 to D84, D87 to D85, D88 to D86, D30 to D87, D89 to D88, D91 to D89, D6 to D9, D92 to D90, D36 to D91, D48 to D92, D54 to D93, D60 to D94, MX92 to MX1, MX94 to MX10, MX15 to MX100, MX32 to MX101, MX49 to MX102, MX89 to MX103, MX16 to MX104, MX33 to MX105, MX50 to MX106, MX88 to MX107, MX90 to MX108, MX17 to MX109, MX2 to MX11, MX34 to MX110, MX51 to MX111, MX91 to MX112, MX19 to MX12, MX36 to MX13, MX53 to MX14, MX67 to MX15, MX81 to MX16, MX93 to MX17, MX105 to MX18, MX20 to MX19, MX1 to MX2, MX37 to MX20, MX54 to MX21, MX68 to MX22, MX82 to MX23, MX3 to MX24, MX106 to MX25, MX21 to MX26, MX38 to MX27, MX55 to MX28, MX69 to MX29, MX18 to MX3, MX4 to MX30, MX107 to MX31, MX22 to MX32, MX39 to MX33, MX56 to MX34, MX70 to MX35, MX5 to MX36, MX108 to MX37, MX6 to MX38, MX23 to MX39, MX35 to MX4, MX57 to MX41, MX71 to MX42, MX95 to MX43, MX7 to MX44, MX24 to MX45, MX41 to MX46, MX58 to MX47, MX72 to MX48, MX83 to MX49, MX101 to MX5, MX8 to MX50, MX25 to MX51, MX42 to MX52, MX59 to MX53, MX73 to MX54, MX9 to MX55, MX26 to MX56, MX43 to MX57, MX60 to MX58, MX74 to MX59, MX66 to MX6, MX112 to MX60, MX27 to MX61, MX44 to MX62, MX61 to MX63, MX75 to MX64, MX10 to MX65, MX11 to MX66, MX28 to MX67, MX45 to MX68, MX62 to MX69, MX102 to MX7, MX76 to MX70, MX84 to MX71, MX113 to MX72, MX96 to MX73, MX12 to MX74, MX29 to MX75, MX46 to MX76, MX63 to MX77, MX77 to MX78, MX85 to MX79, MX80 to MX8, MX114 to MX80, MX97 to MX81, MX13 to MX82, MX30 to MX83, MX47 to MX84, MX64 to MX85, MX103 to MX86, MX78 to MX87, MX86 to MX88, MX115 to MX89, MX52 to MX9, MX99 to MX90, MX98 to MX91, MX14 to MX92, MX31 to MX93, MX100 to MX94, MX65 to MX95, MX104 to MX96, MX79 to MX97, MX87 to MX98, MX48 to MX99, R3 to R1, R2 to R10, R8 to R2, R9 to R3, R7 to R6, R5 to R7, R6 to R8, R1 to R9, USB2 to USB1, USB1 to USB2
Connections:
- net at U1.41 (PF0): now also R5.2
- new net RGB: R5.1
