File: Salane Reboot/Paranoid/TKL/Atmega32U4/Solder Main Branch/RGB Strip.sch (KiCad schematic (older format))
At the start: 1 part

Commit message: a
Parts:
- added C10, C11, C12, C13, C14, C15, C16, C17, C18, C19, C20, C21, C22, C23, C24, C25, C26, C27, C28, C9: 0.1uF, sanproject-keyboard-part:C_0603, symbol Device:C_Small
- added RGB1, RGB10, RGB11, RGB12, RGB13, RGB14, RGB15, RGB16, RGB17, RGB18, RGB19, RGB2, RGB20, RGB21, RGB22, RGB23, RGB24, RGB25, RGB26, RGB27, RGB28, RGB29, RGB3, RGB30, RGB5, RGB6, RGB7, RGB8, RGB9: WS2812B, sanproject-keyboard-part:LED_SK6812MINI_PLCC4_3.5x3.5mm_P1.75mm, symbol LED:WS2812B
- RGB4: renamed from RGB; value SK6812MINI -> WS2812B; footprint LED_SMD:LED_SK6812MINI_PLCC4_3.5x3.5mm_P1.75mm -> sanproject-keyboard-part:LED_SK6812MINI_PLCC4_3.5x3.5mm_P1.75mm; symbol LED:SK6812MINI -> LED:WS2812B
Connections:
- net +5V: now reaches RGB4.1 (VDD)
- net +5V: now also RGB1.1 (VDD), RGB10.1 (VDD), RGB11.1 (VDD), RGB12.1 (VDD), RGB13.1 (VDD), RGB14.1 (VDD), RGB15.1 (VDD), RGB16.1 (VDD), RGB17.1 (VDD), RGB18.1 (VDD), RGB19.1 (VDD), RGB2.1 (VDD), RGB20.1 (VDD), RGB21.1 (VDD), RGB22.1 (VDD), RGB23.1 (VDD), RGB24.1 (VDD), RGB25.1 (VDD), RGB26.1 (VDD), RGB27.1 (VDD), RGB28.1 (VDD), RGB29.1 (VDD), RGB3.1 (VDD), RGB30.1 (VDD), RGB5.1 (VDD), RGB6.1 (VDD), RGB7.1 (VDD), RGB8.1 (VDD), RGB9.1 (VDD)
- net at RGB4.2 (DOUT): now also RGB7.4 (DIN)
- net GND: now reaches RGB4.3 (VSS)
- net GND: now also RGB1.3 (VSS), RGB10.3 (VSS), RGB11.3 (VSS), RGB12.3 (VSS), RGB13.3 (VSS), RGB14.3 (VSS), RGB15.3 (VSS), RGB16.3 (VSS), RGB17.3 (VSS), RGB18.3 (VSS), RGB19.3 (VSS), RGB2.3 (VSS), RGB20.3 (VSS), RGB21.3 (VSS), RGB22.3 (VSS), RGB23.3 (VSS), RGB24.3 (VSS), RGB25.3 (VSS), RGB26.3 (VSS), RGB27.3 (VSS), RGB28.3 (VSS), RGB29.3 (VSS), RGB3.3 (VSS), RGB30.3 (VSS), RGB5.3 (VSS), RGB6.3 (VSS), RGB7.3 (VSS), RGB8.3 (VSS), RGB9.3 (VSS)
- net at RGB4.4 (DIN): now also RGB1.2 (DOUT)
- new net: RGB10.4 (DIN), RGB7.2 (DOUT)
- new net: RGB10.2 (DOUT), RGB13.4 (DIN)
- new net: RGB2.2 (DOUT), RGB5.4 (DIN)
- new net: RGB5.2 (DOUT), RGB8.4 (DIN)
- new net: RGB11.4 (DIN), RGB8.2 (DOUT)
- new net: RGB11.2 (DOUT), RGB14.4 (DIN)
- new net: RGB14.2 (DOUT), RGB15.4 (DIN)
- new net: RGB15.2 (DOUT), RGB16.4 (DIN)
- new net: RGB16.2 (DOUT), RGB17.4 (DIN)
- new net: RGB17.2 (DOUT), RGB18.4 (DIN)
- new net: RGB18.2 (DOUT), RGB19.4 (DIN)
- new net: RGB20.2 (DOUT), RGB3.4 (DIN)
- new net: RGB3.2 (DOUT), RGB6.4 (DIN)
- new net: RGB6.2 (DOUT), RGB9.4 (DIN)
- new net: RGB12.4 (DIN), RGB9.2 (DOUT)
- new net: RGB21.2 (DOUT), RGB22.4 (DIN)
- new net: RGB22.2 (DOUT), RGB23.4 (DIN)
- new net: RGB23.2 (DOUT), RGB24.4 (DIN)
- new net: RGB24.2 (DOUT), RGB25.4 (DIN)
- new net: RGB25.2 (DOUT), RGB26.4 (DIN)
- new net: RGB26.2 (DOUT), RGB27.4 (DIN)
- new net: RGB27.2 (DOUT), RGB28.4 (DIN)
- new net: RGB28.2 (DOUT), RGB29.4 (DIN)
- new net: RGB29.2 (DOUT), RGB30.4 (DIN)
- new net Strip1: RGB13.2 (DOUT), RGB2.4 (DIN)
- new net Strip2: RGB19.2 (DOUT), RGB20.4 (DIN)
- new net Strip3: RGB12.2 (DOUT), RGB21.4 (DIN)
Other:
- moved on the sheet: RGB4

Commit message: a
Connections:
- net +5V: now also C10.2, C11.2, C12.2, C13.2, C14.2, C15.2, C16.2, C17.2, C18.2, C19.1, C20.1, C21.1, C22.1, C23.1, C24.1, C25.1, C26.1, C27.1, C28.1, C9.2
- net GND: now also C10.1, C11.1, C12.1, C13.1, C14.1, C15.1, C16.1, C17.1, C18.1, C19.2, C20.2, C21.2, C22.2, C23.2, C24.2, C25.2, C26.2, C27.2, C28.2, C9.1
Changed lines of the file:
@@
 Connection ~ 5450 750
 $Comp
-L power:+5V #PWR?
+L power:+5V #PWR0101
 U 1 1 639BB63D
 P 5750 750
-F 0 "#PWR?" H 5750 600 50  0001 C CNN
+F 0 "#PWR0101" H 5750 600 50  0001 C CNN
 F 1 "+5V" V 5765 878 50  0000 L CNN
 F 2 "" H 5750 750 50  0001 C CNN
@@
 $EndComp
 $Comp
-L power:GND #PWR?
+L power:GND #PWR0102
 U 1 1 639BC16C
 P 5750 1350
-F 0 "#PWR?" H 5750 1100 50  0001 C CNN
+F 0 "#PWR0102" H 5750 1100 50  0001 C CNN
 F 1 "GND" V 5755 1222 50  0000 R CNN
 F 2 "" H 5750 1350 50  0001 C CNN
@@
 	10950 1500 11250 1500
 $Comp
-L power:+5V #PWR?
+L power:+5V #PWR0103
 U 1 1 639BD6DD
 P 11250 1500
-F 0 "#PWR?" H 11250 1350 50  0001 C CNN
+F 0 "#PWR0103" H 11250 1350 50  0001 C CNN
 F 1 "+5V" V 11265 1628 50  0000 L CNN
 F 2 "" H 11250 1500 50  0001 C CNN
@@
 $EndComp
 $Comp
-L power:GND #PWR?
+L power:GND #PWR0104
 U 1 1 639BD6E3
 P 11250 2100
-F 0 "#PWR?" H 11250 1850 50  0001 C CNN
+F 0 "#PWR0104" H 11250 1850 50  0001 C CNN
 F 1 "GND" V 11255 1972 50  0000 R CNN
 F 2 "" H 11250 2100 50  0001 C CNN
@@
 	5450 2250 5750 2250
 $Comp
-L power:+5V #PWR?
+L power:+5V #PWR0105
 U 1 1 639C6C37
 P 5750 2250
-F 0 "#PWR?" H 5750 2100 50  0001 C CNN
+F 0 "#PWR0105" H 5750 2100 50  0001 C CNN
 F 1 "+5V" V 5765 2378 50  0000 L CNN
 F 2 "" H 5750 2250 50  0001 C CNN
@@
 $EndComp
 $Comp
-L power:GND #PWR?
+L power:GND #PWR0106
 U 1 1 639C6C3D
 P 5750 2850
-F 0 "#PWR?" H 5750 2600 50  0001 C CNN
+F 0 "#PWR0106" H 5750 2600 50  0001 C CNN
 F 1 "GND" V 5755 2722 50  0000 R CNN
 F 2 "" H 5750 2850 50  0001 C CNN
@@
 	10950 3000 11250 3000
 $Comp
-L power:+5V #PWR?
+L power:+5V #PWR0107
 U 1 1 639E0E89
 P 11250 3000
-F 0 "#PWR?" H 11250 2850 50  0001 C CNN
+F 0 "#PWR0107" H 11250 2850 50  0001 C CNN
 F 1 "+5V" V 11265 3128 50  0000 L CNN
 F 2 "" H 11250 3000 50  0001 C CNN
@@
 $EndComp
 $Comp
-L power:GND #PWR?
+L power:GND #PWR0108
 U 1 1 639E0E8F
 P 11250 3600
-F 0 "#PWR?" H 11250 3350 50  0001 C CNN
+F 0 "#PWR0108" H 11250 3350 50  0001 C CNN
 F 1 "GND" V 11255 3472 50  0000 R CNN
 F 2 "" H 11250 3600 50  0001 C CNN
@@
 Connection ~ 10950 3000
 Connection ~ 10950 3600
+Wire Wire Line
+	1450 4650 1850 4650
+Connection ~ 1850 4650
+Wire Wire Line
+	1850 4650 2250 4650
+Connection ~ 2250 4650
+Wire Wire Line
+	2250 4650 2650 4650
+Connection ~ 2650 4650
+Wire Wire Line
+	2650 4650 3050 4650
+Connection ~ 3050 4650
+Wire Wire Line
+	3050 4650 3450 4650
+Connection ~ 3450 4650
+Wire Wire Line
+	3450 4650 3850 4650
+Connection ~ 3850 4650
+Wire Wire Line
+	3850 4650 4250 4650
+Connection ~ 4250 4650
+Wire Wire Line
+	4250 4650 4650 4650
+Connection ~ 4650 4650
+Wire Wire Line
+	4650 4650 5050 4650
+Wire Wire Line
+	1450 4850 1850 4850
+Connection ~ 1850 4850
+Wire Wire Line
+	1850 4850 2250 4850
+Connection ~ 2250 4850
+Wire Wire Line
+	2250 4850 2650 4850
+Connection ~ 2650 4850
+Wire Wire Line
+	2650 4850 3050 4850
+Connection ~ 3050 4850
+Wire Wire Line
+	3050 4850 3450 4850
+Connection ~ 3450 4850
+Wire Wire Line
+	3450 4850 3850 4850
+Connection ~ 3850 4850
+Wire Wire Line
+	3850 4850 4250 4850
+Connection ~ 4250 4850
+Wire Wire Line
+	4250 4850 4650 4850
+Connection ~ 4650 4850
+Wire Wire Line
+	4650 4850 5050 4850
+Wire Wire Line
+	1450 5000 1850 5000
+Connection ~ 1850 5000
+Wire Wire Line
+	1850 5000 2250 5000
+Connection ~ 2250 5000
+Wire Wire Line
+	2250 5000 2650 5000
+Connection ~ 2650 5000
+Wire Wire Line
+	2650 5000 3050 5000
+Connection ~ 3050 5000
+Wire Wire Line
+	3050 5000 3450 5000
+Connection ~ 3450 5000
+Wire Wire Line
+	3450 5000 3850 5000
+Connection ~ 3850 5000
+Wire Wire Line
+	3850 5000 4250 5000
+Connection ~ 4250 5000
+Wire Wire Line
+	4250 5000 4650 5000
+Connection ~ 4650 5000
+Wire Wire Line
+	4650 5000 5050 5000
+Wire Wire Line
+	1450 5200 1850 5200
+Connection ~ 1850 5200
+Wire Wire Line
+	1850 5200 2250 5200
+Connection ~ 2250 5200
+Wire Wire Line
+	2250 5200 2650 5200
+Connection ~ 2650 5200
+Wire Wire Line
+	2650 5200 3050 5200
+Connection ~ 3050 5200
+Wire Wire Line
+	3050 5200 3450 5200
+Connection ~ 3450 5200
+Wire Wire Line
+	3450 5200 3850 5200
+Connection ~ 3850 5200
+Wire Wire Line
+	3850 5200 4250 5200
+Connection ~ 4250 5200
+Wire Wire Line
+	4250 5200 4650 5200
+Connection ~ 4650 5200
+Wire Wire Line
+	4650 5200 5050 5200
+Wire Wire Line
+	1450 4650 1250 4650
+Connection ~ 1450 4650
+Wire Wire Line
+	1450 4850 1250 4850
+Connection ~ 1450 4850
+$Comp
+L power:GND #PWR0109
+U 1 1 63849908
+P 1250 4650
+F 0 "#PWR0109" H 1250 4400 50  0001 C CNN
+F 1 "GND" V 1255 4522 50  0000 R CNN
+F 2 "" H 1250 4650 50  0001 C CNN
+F 3 "" H 1250 4650 50  0001 C CNN
+	1    1250 4650
+	0    1    1    0
+$EndComp
+$Comp
+L power:+5V #PWR0110
+U 1 1 63849EA3
+P 1250 4850
+F 0 "#PWR0110" H 1250 4700 50  0001 C CNN
+F 1 "+5V" V 1265 4978 50  0000 L CNN
+F 2 "" H 1250 4850 50  0001 C CNN
+F 3 "" H 1250 4850 50  0001 C CNN
+	1    1250 4850
+	0    -1   -1   0
+$EndComp
+Wire Wire Line
+	1450 5000 1250 5000
+Wire Wire Line
+	1450 5200 1250 5200
+$Comp
+L power:GND #PWR0111
+U 1 1 638A52EB
+P 1250 5200
+F 0 "#PWR0111" H 1250 4950 50  0001 C CNN
+F 1 "GND" V 1255 5072 50  0000 R CNN
+F 2 "" H 1250 5200 50  0001 C CNN
+F 3 "" H 1250 5200 50  0001 C CNN
+	1    1250 5200
+	0    1    1    0
+$EndComp
+$Comp
+L power:+5V #PWR0112
+U 1 1 638A52F1
+P 1250 5000
+F 0 "#PWR0112" H 1250 4850 50  0001 C CNN
+F 1 "+5V" V 1265 5128 50  0000 L CNN
+F 2 "" H 1250 5000 50  0001 C CNN
+F 3 "" H 1250 5000 50  0001 C CNN
+	1    1250 5000
+	0    -1   -1   0
+$EndComp
+Connection ~ 1450 5000
+Connection ~ 1450 5200
 $EndSCHEMATC
