File: Salane Reboot/Paranoid/TKL/Atmega32U4/Solder Main Branch/Solder - Copy.kicad_pcb (KiCad board)
At the start: 2 copper layers, 344 x 124 mm, 282 parts, among them J1 Conn_01x06_Female, J2 Conn_01x04_Female, U1 ATmega32U4-MU, U2 PRTR5V0U2X, Y1 16MHz

Commit message: a
Parts:
- moved D9 26.2 mm to (75.3, 134.7)
Routing:
- net Net-(RGB20-Pad2): track 1.21 -> 19.9 mm
- net Net-(RGB3-Pad2): track 0.00 -> 16.9 mm
- net R10: track 367.6 -> 368.4 mm
