File: KiCad/Daughterboard/AI03 USB daughterboard/Unified-Daughterboard-master/KiCad/C3/Unified-Daughterboard.kicad_pcb (KiCad board)
At the start: 2 copper layers, 98 x 107.5 mm, 354 parts, among them J1 TYPE-C-31-M12_13, J2 SM04B-SRSS-TB(LF)(SN), U1 TPD4E05U06DQAR

Commit message: a
Parts:
- removed the J1 at (75.0, 138.8)
- removed the J1 at (75.0, 120.3)
- removed the J1 at (75.0, 101.8)
- removed the J1 at (75.0, 83.3)
- removed the J1 at (75.0, 64.8)
- removed the REF** at (154.0, 152.0)
- removed the REF** at (76.0, 152.0)
- removed the REF** at (154.0, 51.5)
- removed the REF** at (76.0, 51.5)
- removed the mouse-bite-3mm-slot at (115.0, 147.8)
- removed the mouse-bite-3mm-slot at (75.0, 55.8)
- removed the mouse-bite-3mm-slot at (135.0, 147.8)
- removed the mouse-bite-3mm-slot at (155.0, 147.8)
- removed the mouse-bite-3mm-slot at (95.0, 147.8)
- removed the mouse-bite-3mm-slot at (75.0, 147.8)
- removed the mouse-bite-3mm-slot at (155.0, 55.8)
- removed the mouse-bite-3mm-slot at (135.0, 55.8)
- removed the mouse-bite-3mm-slot at (115.0, 55.8)
- removed the mouse-bite-3mm-slot at (95.0, 55.8)
- added G***: LOGO, logo:salane mini, B.Cu at (155.0, 140.0)
- added G***: LOGO, logo:salane mini, B.Cu at (75.0, 121.5)
- added G***: LOGO, logo:salane mini, B.Cu at (155.0, 103.0)
- added G***: LOGO, logo:salane mini, B.Cu at (135.0, 103.0)
- added G***: LOGO, logo:salane mini, B.Cu at (115.0, 103.0)
- added G***: LOGO, logo:salane mini, B.Cu at (95.0, 103.0)
- added G***: LOGO, logo:salane mini, B.Cu at (75.0, 103.0)
- added G***: LOGO, logo:salane mini, B.Cu at (155.0, 84.5)
- added G***: LOGO, logo:salane mini, B.Cu at (135.0, 84.5)
- added G***: LOGO, logo:salane mini, B.Cu at (115.0, 84.5)
- added G***: LOGO, logo:salane mini, B.Cu at (95.0, 84.5)
- added G***: LOGO, logo:salane mini, B.Cu at (135.0, 140.0)
- added G***: LOGO, logo:salane mini, B.Cu at (75.0, 84.5)
- added G***: LOGO, logo:salane mini, B.Cu at (155.0, 66.0)
- added G***: LOGO, logo:salane mini, B.Cu at (135.0, 66.0)
- added G***: LOGO, logo:salane mini, B.Cu at (115.0, 66.0)
- added G***: LOGO, logo:salane mini, B.Cu at (95.0, 66.0)
- added G***: LOGO, logo:salane mini, B.Cu at (75.0, 66.0)
- added G***: LOGO, logo:salane mini, B.Cu at (115.0, 140.0)
- added G***: LOGO, logo:salane mini, B.Cu at (95.0, 140.0)
- added G***: LOGO, logo:salane mini, B.Cu at (75.0, 140.0)
- added G***: LOGO, logo:salane mini, B.Cu at (155.0, 121.5)
- added G***: LOGO, logo:salane mini, B.Cu at (135.0, 121.5)
- added G***: LOGO, logo:salane mini, B.Cu at (115.0, 121.5)
- added G***: LOGO, logo:salane mini, B.Cu at (95.0, 121.5)
- added J1: TYPE-C-31-M12_13, sanproject-keyboard-part:TYPE-C-31-M-12, F.Cu at (75.0, 64.8)
- added J1: TYPE-C-31-M12_13, sanproject-keyboard-part:TYPE-C-31-M-12, F.Cu at (75.0, 120.3)
- added J1: TYPE-C-31-M12_13, sanproject-keyboard-part:TYPE-C-31-M-12, F.Cu at (75.0, 83.3)
- added J1: TYPE-C-31-M12_13, sanproject-keyboard-part:TYPE-C-31-M-12, F.Cu at (75.0, 138.8)
- added J1: TYPE-C-31-M12_13, sanproject-keyboard-part:TYPE-C-31-M-12, F.Cu at (75.0, 101.8)
- added REF**: 1mm origin reel, sanproject-keyboard-part:OriginPoint, F.Cu at (169.5, 66.5)
- added REF**: 1mm origin reel, sanproject-keyboard-part:OriginPoint, F.Cu at (169.5, 137.0)
- added REF**: 1mm origin reel, sanproject-keyboard-part:OriginPoint, F.Cu at (60.5, 66.5)
- added REF**: 1mm origin reel, sanproject-keyboard-part:OriginPoint, F.Cu at (60.5, 137.0)
- added mouse-bite-3mm-slot: VAL**, sanproject-keyboard-part:mouse-bite-3mm-slot-half, F.Cu at (165.0, 138.8)
- added mouse-bite-3mm-slot: VAL**, sanproject-keyboard-part:mouse-bite-3mm-slot-half, F.Cu at (65.0, 64.8)
- added mouse-bite-3mm-slot: VAL**, sanproject-keyboard-part:mouse-bite-3mm-slot-half, F.Cu at (165.0, 120.3)
- added mouse-bite-3mm-slot: VAL**, sanproject-keyboard-part:mouse-bite-3mm-slot-half, F.Cu at (165.0, 101.8)
- added mouse-bite-3mm-slot: VAL**, sanproject-keyboard-part:mouse-bite-3mm-slot-half, F.Cu at (165.0, 83.3)
- added mouse-bite-3mm-slot: VAL**, sanproject-keyboard-part:mouse-bite-3mm-slot-half, F.Cu at (165.0, 64.8)
- added mouse-bite-3mm-slot: VAL**, sanproject-keyboard-part:mouse-bite-3mm-slot-half, F.Cu at (65.0, 138.8)
- added mouse-bite-3mm-slot: VAL**, sanproject-keyboard-part:mouse-bite-3mm-slot-half, F.Cu at (65.0, 120.3)
- added mouse-bite-3mm-slot: VAL**, sanproject-keyboard-part:mouse-bite-3mm-slot-half, F.Cu at (65.0, 101.8)
- added mouse-bite-3mm-slot: VAL**, sanproject-keyboard-part:mouse-bite-3mm-slot-half, F.Cu at (65.0, 83.3)
- J1 (x20): footprint acheron_Connectors:TYPE-C-31-M-12 -> sanproject-keyboard-part:TYPE-C-31-M-12
Other:
- board size 98 x 107.5 mm -> 116 x 90.5 mm
