File: Salane Reboot/Paranoid/TKL/Atmega32U4/Solder/Solder.kicad_pcb (KiCad board)
At the start: 2 copper layers, 344 x 124 mm, 296 parts, among them J1 Conn_01x06_Female, J2 Suit, J3 HIney/Mechlovin, J4 Breakout, J5 Amber TKL, SW1 SW_Push, U1 ATmega32U4-MU, U2 PRTR5V0U2X, Y1 16MHz

Commit message: a
Parts:
- added G***: LOGO, logo:SalaneReboot, F.Cu at (345.6, 95.1)
- added G***: LOGO, logo:Paranoid, B.Cu at (337.3, 94.0)
- added J6: RGB JST, sanproject-keyboard-part:JST-SR-3, B.Cu at (358.6, 117.8)
- added J7: RGB Breakout, sanproject-keyboard-part:RGB-Header, B.Cu at (358.6, 115.4)
- added JP1: Jumper_NC_Dual, sanproject-keyboard-part:SolderJumper-3_P1.3mm_Open_Pad1.0x1.5mm, B.Cu at (48.0, 123.7)
Connections:
- RGB1 pad 4: RGB -> Underglow
Routing:
- net (no net): track 329.0 -> 2.86 mm, vias 1 -> 0
- net DOUT: track 0.00 -> 323.1 mm, vias 0 -> 1
- net Underglow: track 0.00 -> 22.5 mm, vias 0 -> 2
- net Net-(D9-Pad2): track 5.47 -> 16.2 mm
- net +5V: track 1349.8 -> 1358.1 mm
- net GND: track 141.8 -> 149.6 mm
- net RGB: track 33.2 -> 39.8 mm
- net Net-(D81-Pad2): track 5.47 -> 10.6 mm
- net Net-(D75-Pad2): track 5.47 -> 10.6 mm
- net Net-(D69-Pad2): track 5.47 -> 10.6 mm
- net Net-(D21-Pad2): track 5.47 -> 10.6 mm
Other:
- outline, holes or cut-outs redrawn
- board text added: "+"
- board text added: "-"
- board text added: "->"
